Commit message: Robot description file updated with inertial elements, in order to work in Gazebo.

File: src/bioloid_master/urdf/bioloid.urdf (robot description, URDF)
Before this commit: robot bioloid, 26 links, 25 joints
Links:
- link imu_link: mass None -> 1.0
- link left_ankle_lateral_link: mass None -> 1.0
- link left_ankle_swing_link: mass None -> 1.0
- link left_foot_link: mass None -> 1.0
- link left_hand_link: mass None -> 1.0
- link left_hip_lateral_link: mass None -> 1.0
- link left_hip_twist_link: mass None -> 1.0
- link left_lower_arm_link: mass None -> 1.0
- link left_lower_leg_link: mass None -> 1.0
- link left_shoulder_swing_link: mass None -> 1.0
- link left_upper_arm_link: mass None -> 1.0
- link left_upper_leg_link: mass None -> 1.0
- link right_ankle_lateral_link: mass None -> 1.0
- link right_ankle_swing_link: mass None -> 1.0
- link right_foot_link: mass None -> 1.0
- link right_hand_link: mass None -> 1.0
- link right_hip_lateral_link: mass None -> 1.0
- link right_hip_twist_link: mass None -> 1.0
- link right_lower_arm_link: mass None -> 1.0
- link right_lower_leg_link: mass None -> 1.0
- link right_shoulder_swing_link: mass None -> 1.0
- link right_upper_arm_link: mass None -> 1.0
- link right_upper_leg_link: mass None -> 1.0
- link torso_link: mass None -> 1.0
Joints:
- joint left_knee_joint: limit lower=-3.14159 upper=0 effort=10 velocity=1.0 -> lower=-3.14159 upper=0.0 effort=10 velocity=1.0
- joint right_knee_joint: limit lower=-3.14159 upper=0 effort=10 velocity=1.0 -> lower=-3.14159 upper=0.0 effort=10 velocity=1.0

File: src/bioloid_master/urdf/bioloid.xacro (robot description, xacro)
@@ -121,4 +121,9 @@
         </material>
     </visual>
+    <inertial>
+      <origin xyz="0 0 0"/>
+      <mass value="1.0"/>
+      <inertia  ixx="0.001" ixy="0.0"  ixz="0.0"  iyy="0.001"  iyz="0.0"  izz="0.001"/>
+    </inertial>
 </link>
 <!-- Base -->
@@ -144,5 +149,10 @@
             <color rgba="0.0 0.0 0.0 1.0"/>
         </material>
-    </visual>-->
+    </visual>
+    <inertial>
+      <origin xyz="0 0 0"/>
+      <mass value="1.0"/>
+      <inertia  ixx="0.001" ixy="0.0"  ixz="0.0"  iyy="0.001"  iyz="0.0"  izz="0.001"/>
+    </inertial>-->
 </link>
 <!-- Torso -->
@@ -211,4 +221,9 @@
         </geometry>
     </collision>
+    <inertial>
+      <origin xyz="0 0 0"/>
+      <mass value="1.0"/>
+      <inertia  ixx="0.001" ixy="0.0"  ixz="0.0"  iyy="0.001"  iyz="0.0"  izz="0.001"/>
+    </inertial>
 </link>
 <!-- Torso to right shoulder -->
@@ -225,4 +240,9 @@
         </geometry>
     </collision>
+    <inertial>
+      <origin xyz="0 0 0"/>
+      <mass value="1.0"/>
+      <inertia  ixx="0.001" ixy="0.0"  ixz="0.0"  iyy="0.001"  iyz="0.0"  izz="0.001"/>
+    </inertial>
 </link>
 <!-- Torso to left shoulder -->
@@ -239,4 +259,9 @@
         </geometry>
     </collision>
+    <inertial>
+      <origin xyz="0 0 0"/>
+      <mass value="1.0"/>
+      <inertia  ixx="0.001" ixy="0.0"  ixz="0.0"  iyy="0.001"  iyz="0.0"  izz="0.001"/>
+    </inertial>
 </link>
 <!-- Right shoulder to upper arm -->
@@ -275,4 +300,9 @@
         </geometry>
     </collision>
+    <inertial>
+      <origin xyz="0 0 0"/>
+      <mass value="1.0"/>
+      <inertia  ixx="0.001" ixy="0.0"  ixz="0.0"  iyy="0.001"  iyz="0.0"  izz="0.001"/>
+    </inertial>
 </link>
 <!-- Left shoulder to upper arm -->
@@ -311,4 +341,9 @@
         </geometry>
     </collision>
+    <inertial>
+      <origin xyz="0 0 0"/>
+      <mass value="1.0"/>
+      <inertia  ixx="0.001" ixy="0.0"  ixz="0.0"  iyy="0.001"  iyz="0.0"  izz="0.001"/>
+    </inertial>
 </link>
 <!-- Right upper arm to lower arm -->
@@ -338,4 +373,9 @@
         </geometry>
     </collision>
+    <inertial>
+      <origin xyz="0 0 0"/>
+      <mass value="1.0"/>
+      <inertia  ixx="0.001" ixy="0.0"  ixz="0.0"  iyy="0.001"  iyz="0.0"  izz="0.001"/>
+    </inertial>
 </link>
 <!-- Right lower arm to hand -->
@@ -358,4 +398,9 @@
         </geometry>
     </collision>
+    <inertial>
+      <origin xyz="0 0 0"/>
+      <mass value="1.0"/>
+      <inertia  ixx="0.001" ixy="0.0"  ixz="0.0"  iyy="0.001"  iyz="0.0"  izz="0.001"/>
+    </inertial>
 </link>
 <!-- Left upper arm to lower arm -->
@@ -385,4 +430,9 @@
         </geometry>
     </collision>
+    <inertial>
+      <origin xyz="0 0 0"/>
+      <mass value="1.0"/>
+      <inertia  ixx="0.001" ixy="0.0"  ixz="0.0"  iyy="0.001"  iyz="0.0"  izz="0.001"/>
+    </inertial>
 </link>
 <!-- Left lower arm to hand -->
@@ -405,4 +455,9 @@
         </geometry>
     </collision>
+    <inertial>
+      <origin xyz="0 0 0"/>
+      <mass value="1.0"/>
+      <inertia  ixx="0.001" ixy="0.0"  ixz="0.0"  iyy="0.001"  iyz="0.0"  izz="0.001"/>
+    </inertial>
 </link>
 <!-- Torso to right hip twist -->
@@ -419,4 +474,9 @@
         </geometry>
     </collision>
+    <inertial>
+      <origin xyz="0 0 0"/>
+      <mass value="1.0"/>
+      <inertia  ixx="0.001" ixy="0.0"  ixz="0.0"  iyy="0.001"  iyz="0.0"  izz="0.001"/>
+    </inertial>
 </link>
 <!-- Torso to left hip twist -->
@@ -433,4 +493,9 @@
         </geometry>
     </collision>
+    <inertial>
+      <origin xyz="0 0 0"/>
+      <mass value="1.0"/>
+      <inertia  ixx="0.001" ixy="0.0"  ixz="0.0"  iyy="0.001"  iyz="0.0"  izz="0.001"/>
+    </inertial>
 </link>
 <!-- Right hip twist to hip lateral -->
@@ -469,4 +534,9 @@
         </geometry>
     </collision>
+    <inertial>
+      <origin xyz="0 0 0"/>
+      <mass value="1.0"/>
+      <inertia  ixx="0.001" ixy="0.0"  ixz="0.0"  iyy="0.001"  iyz="0.0"  izz="0.001"/>
+    </inertial>
 </link>
 <!-- Left hip twist to hip lateral -->
@@ -505,4 +575,9 @@
         </geometry>
     </collision>
+    <inertial>
+      <origin xyz="0 0 0"/>
+      <mass value="1.0"/>
+      <inertia  ixx="0.001" ixy="0.0"  ixz="0.0"  iyy="0.001"  iyz="0.0"  izz="0.001"/>
+    </inertial>
 </link>
 <!-- Right hip lateral to upper leg -->
@@ -529,4 +604,9 @@
         </geometry>
     </collision>
+    <inertial>
+      <origin xyz="0 0 0"/>
+      <mass value="1.0"/>
+      <inertia  ixx="0.001" ixy="0.0"  ixz="0.0"  iyy="0.001"  iyz="0.0"  izz="0.001"/>
+    </inertial>
 </link>
 <!-- Left hip lateral to upper leg -->
@@ -553,4 +633,9 @@
         </geometry>
     </collision>
+    <inertial>
+      <origin xyz="0 0 0"/>
+      <mass value="1.0"/>
+      <inertia  ixx="0.001" ixy="0.0"  ixz="0.0"  iyy="0.001"  iyz="0.0"  izz="0.001"/>
+    </inertial>
 </link>
 <!-- Right upper leg to lower leg -->
@@ -582,4 +667,9 @@
         </geometry>
     </collision>
+    <inertial>
+      <origin xyz="0 0 0"/>
+      <mass value="1.0"/>
+      <inertia  ixx="0.001" ixy="0.0"  ixz="0.0"  iyy="0.001"  iyz="0.0"  izz="0.001"/>
+    </inertial>
 </link>
 <!-- Left upper leg to lower leg -->
@@ -611,4 +701,9 @@
         </geometry>
     </collision>
+    <inertial>
+      <origin xyz="0 0 0"/>
+      <mass value="1.0"/>
+      <inertia  ixx="0.001" ixy="0.0"  ixz="0.0"  iyy="0.001"  iyz="0.0"  izz="0.001"/>
+    </inertial>
 </link>
 <!-- Right lower leg to ankle swing -->
@@ -643,4 +738,9 @@
         </geometry>
     </collision>
+    <inertial>
+      <origin xyz="0 0 0"/>
+      <mass value="1.0"/>
+      <inertia  ixx="0.001" ixy="0.0"  ixz="0.0"  iyy="0.001"  iyz="0.0"  izz="0.001"/>
+    </inertial>
 </link>
 <!-- Left lower leg to ankle swing -->
@@ -675,4 +775,9 @@
         </geometry>
     </collision>
+    <inertial>
+      <origin xyz="0 0 0"/>
+      <mass value="1.0"/>
+      <inertia  ixx="0.001" ixy="0.0"  ixz="0.0"  iyy="0.001"  iyz="0.0"  izz="0.001"/>
+    </inertial>
 </link>
 <!-- Right ankle swing to ankle lateral -->
@@ -693,4 +798,9 @@
         </geometry>
     </collision>
+    <inertial>
+      <origin xyz="0 0 0"/>
+      <mass value="1.0"/>
+      <inertia  ixx="0.001" ixy="0.0"  ixz="0.0"  iyy="0.001"  iyz="0.0"  izz="0.001"/>
+    </inertial>
 </link>
 <!-- Right ankle lateral to foot -->
@@ -707,4 +817,9 @@
         </geometry>
     </collision>
+    <inertial>
+      <origin xyz="0 0 0"/>
+      <mass value="1.0"/>
+      <inertia  ixx="0.001" ixy="0.0"  ixz="0.0"  iyy="0.001"  iyz="0.0"  izz="0.001"/>
+    </inertial>
 </link>
 <!-- Left ankle swing to ankle lateral -->
@@ -725,4 +840,9 @@
         </geometry>
     </collision>
+    <inertial>
+      <origin xyz="0 0 0"/>
+      <mass value="1.0"/>
+      <inertia  ixx="0.001" ixy="0.0"  ixz="0.0"  iyy="0.001"  iyz="0.0"  izz="0.001"/>
+    </inertial>
 </link>
 <!-- Left ankle lateral to foot -->
@@ -739,4 +859,9 @@
         </geometry>
     </collision>
+    <inertial>
+      <origin xyz="0 0 0"/>
+      <mass value="1.0"/>
+      <inertia  ixx="0.001" ixy="0.0"  ixz="0.0"  iyy="0.001"  iyz="0.0"  izz="0.001"/>
+    </inertial>
 </link>
 </robot>

Commit message: Zeroed position offsets in joint controller (to be removed completely) Edited URDF and SRDF files so that robot uses default Bioloid home position (arms outstretched) Added ignore path to .gitignore Minor edits

File: src/bioloid_master/urdf/bioloid.urdf (robot description, URDF)
Before this commit: robot bioloid, 27 links, 26 joints
Joints:
- joint left_shoulder_lateral_joint: limit lower=-0.2 upper=3.14159 effort=10 velocity=1.0 -> lower=-3.14159 upper=3.14159 effort=10 velocity=1.0; origin xyz=0.014 0 -0.044 rpy=-1.570795 0 0 -> xyz=0.014 0 -0.044 rpy=-1.570795 1.570795 0
- joint left_shoulder_swing_joint: origin xyz=0.032 0 0 rpy=0 1.570795 3.14159 -> xyz=0.032 0 0 rpy=1.570795 0 -1.570795
- joint right_shoulder_lateral_joint: limit lower=-0.2 upper=3.14159 effort=10 velocity=1.0 -> lower=-3.14159 upper=3.14159 effort=10 velocity=1.0; origin xyz=-0.014 0 0.044 rpy=-1.570795 0 0 -> xyz=-0.014 0 0.044 rpy=-1.570795 1.570795 0
- joint right_shoulder_swing_joint: origin xyz=-0.032 0 0 rpy=0 -1.570795 0.0 -> xyz=-0.032 0 0 rpy=-1.570795 0 1.570795

File: src/bioloid_master/urdf/bioloid.xacro (robot description, xacro)
@@ -13,8 +13,10 @@
     <axis xyz="0 0 1"/>
 </xacro:macro>
-<xacro:macro name="shoulder_swing_joint" params="prefix reflect x">
+<!-- <xacro:macro name="shoulder_swing_joint" params="prefix reflect x"> -->
+<xacro:macro name="shoulder_swing_joint" params="prefix reflect">
     <joint name="${prefix}_shoulder_swing_joint" type="revolute">
         <parent link="torso_link"/>
-        <origin xyz="${reflect*(-0.032)} 0 0" rpy="0 ${reflect*(-pi/2)} ${x*pi}"/>
+        <!-- <origin xyz="${reflect*(-0.032)} 0 0" rpy="0 ${reflect*(-pi/2)} ${x*pi}"/> -->
+        <origin xyz="${reflect*(-0.032)} 0 0" rpy="${reflect*(-pi/2)} 0 ${reflect*(pi/2)}"/>
         <xacro:z_rot/>
         <child link="${prefix}_shoulder_swing_link"/>
@@ -25,8 +27,9 @@
     <joint name="${prefix}_shoulder_lateral_joint" type="revolute">
         <parent link="${prefix}_shoulder_swing_link"/>
-        <origin xyz="${reflect*(-0.014)} 0 ${reflect*0.044}" rpy="${-pi/2} 0 0"/>
+        <!-- <origin xyz="${reflect*(-0.014)} 0 ${reflect*0.044}" rpy="${-pi/2} 0 0"/> -->
+        <origin xyz="${reflect*(-0.014)} 0 ${reflect*0.044}" rpy="${-pi/2} ${pi/2} 0"/>
         <xacro:z_rot/>
         <child link="${prefix}_upper_arm_link"/>
-        <limit lower="${-0.2}" upper="${pi}" effort="10" velocity="1.0"/>
+        <limit lower="${-pi}" upper="${pi}" effort="10" velocity="1.0"/>
     </joint>
 </xacro:macro>
@@ -327,5 +330,5 @@
 </link>
 <!-- Torso to right shoulder -->
-<xacro:shoulder_swing_joint prefix="right" reflect="1" x="0"/>
+<xacro:shoulder_swing_joint prefix="right" reflect="1"/>
 <link name="right_shoulder_swing_link">
     <visual>
@@ -346,5 +349,5 @@
 </link>
 <!-- Torso to left shoulder -->
-<xacro:shoulder_swing_joint prefix="left" reflect="-1" x="1"/>
+<xacro:shoulder_swing_joint prefix="left" reflect="-1"/>
 <link name="left_shoulder_swing_link">
     <visual>

File: src/bioloid_master/urdf/bioloid_compr_18_servos.urdf (robot description, URDF)
Before this commit: robot bioloid_compr_18_servos, 24 links, 23 joints
Joints:
- joint left_shoulder_lateral_joint: limit lower=-0.2 upper=3.14159 effort=10 velocity=1.0 -> lower=-3.14159 upper=3.14159 effort=10 velocity=1.0; origin xyz=0.014 0 -0.044 rpy=-1.570795 0 0 -> xyz=0.014 0 -0.044 rpy=-1.570795 1.570795 0
- joint left_shoulder_swing_joint: origin xyz=0.032 0 0 rpy=0 1.570795 3.14159 -> xyz=0.032 0 0 rpy=1.570795 0 -1.570795
- joint right_shoulder_lateral_joint: limit lower=-0.2 upper=3.14159 effort=10 velocity=1.0 -> lower=-3.14159 upper=3.14159 effort=10 velocity=1.0; origin xyz=-0.014 0 0.044 rpy=-1.570795 0 0 -> xyz=-0.014 0 0.044 rpy=-1.570795 1.570795 0
- joint right_shoulder_swing_joint: origin xyz=-0.032 0 0 rpy=0 -1.570795 0.0 -> xyz=-0.032 0 0 rpy=-1.570795 0 1.570795

File: src/bioloid_master/urdf/bioloid_compr_18_servos.xacro (robot description, xacro)
@@ -13,8 +13,10 @@
     <axis xyz="0 0 1"/>
 </xacro:macro>
-<xacro:macro name="shoulder_swing_joint" params="prefix reflect x">
+<!-- <xacro:macro name="shoulder_swing_joint" params="prefix reflect x"> -->
+<xacro:macro name="shoulder_swing_joint" params="prefix reflect">
     <joint name="${prefix}_shoulder_swing_joint" type="revolute">
         <parent link="torso_link"/>
-        <origin xyz="${reflect*(-0.032)} 0 0" rpy="0 ${reflect*(-pi/2)} ${x*pi}"/>
+        <!-- <origin xyz="${reflect*(-0.032)} 0 0" rpy="0 ${reflect*(-pi/2)} ${x*pi}"/> -->
+        <origin xyz="${reflect*(-0.032)} 0 0" rpy="${reflect*(-pi/2)} 0 ${reflect*(pi/2)}"/>
         <xacro:z_rot/>
         <child link="${prefix}_shoulder_swing_link"/>
@@ -25,8 +27,9 @@
     <joint name="${prefix}_shoulder_lateral_joint" type="revolute">
         <parent link="${prefix}_shoulder_swing_link"/>
-        <origin xyz="${reflect*(-0.014)} 0 ${reflect*0.044}" rpy="${-pi/2} 0 0"/>
+        <!-- <origin xyz="${reflect*(-0.014)} 0 ${reflect*0.044}" rpy="${-pi/2} 0 0"/> -->
+        <origin xyz="${reflect*(-0.014)} 0 ${reflect*0.044}" rpy="${-pi/2} ${pi/2} 0"/>
         <xacro:z_rot/>
         <child link="${prefix}_upper_arm_link"/>
-        <limit lower="${-0.2}" upper="${pi}" effort="10" velocity="1.0"/>
+        <limit lower="${-pi}" upper="${pi}" effort="10" velocity="1.0"/>
     </joint>
 </xacro:macro>
@@ -188,5 +191,5 @@
 </link>
 <!-- Torso to right shoulder -->
-<xacro:shoulder_swing_joint prefix="right" reflect="1" x="0"/>
+<xacro:shoulder_swing_joint prefix="right" reflect="1"/>
 <link name="right_shoulder_swing_link">
     <visual>
@@ -207,5 +210,5 @@
 </link>
 <!-- Torso to left shoulder -->
-<xacro:shoulder_swing_joint prefix="left" reflect="-1" x="1"/>
+<xacro:shoulder_swing_joint prefix="left" reflect="-1"/>
 <link name="left_shoulder_swing_link">
     <visual>

Commit message: Tweaked hip_lateral_joint and hip_swing_joint limits

File: src/bioloid_master/urdf/bioloid.urdf (robot description, URDF)
Before this commit: robot bioloid, 27 links, 26 joints
Joints:
- joint left_hip_lateral_joint: limit lower=-0.3 upper=0.3 effort=10 velocity=1.0 -> lower=-0.3 upper=1.0 effort=10 velocity=1.0
- joint left_hip_swing_joint: limit lower=-1.570795 upper=1.570795 effort=10 velocity=1.0 -> lower=-1.570795 upper=1.9 effort=10 velocity=1.0
- joint right_hip_lateral_joint: limit lower=-0.3 upper=0.3 effort=10 velocity=1.0 -> lower=-0.3 upper=1.0 effort=10 velocity=1.0
- joint right_hip_swing_joint: limit lower=-1.570795 upper=1.570795 effort=10 velocity=1.0 -> lower=-1.570795 upper=1.9 effort=10 velocity=1.0

File: src/bioloid_master/urdf/bioloid.xacro (robot description, xacro)
@@ -73,5 +73,5 @@
             <xacro:z_rot/>
             <child link="${prefix}_hip_lateral_link"/>
-            <limit lower="${-0.3}" upper="${0.3}" effort="10" velocity="1.0"/>
+            <limit lower="${-0.3}" upper="${1.0}" effort="10" velocity="1.0"/>
         </joint>
     </xacro:macro>
@@ -82,5 +82,5 @@
             <xacro:z_rot/>
             <child link="${prefix}_upper_leg_link"/>
-            <limit lower="${-pi/2}" upper="${pi/2}" effort="10" velocity="1.0"/>
+            <limit lower="${-pi/2}" upper="${1.9}" effort="10" velocity="1.0"/>
         </joint>
     </xacro:macro>
