Commit message: Added Gazebo ros_control plugin and transmission elements to URDF. Created gazebo launch and world files. TODO: Find out why Gazebo ros_control plugin fails on startup.

File: src/bioloid_master/urdf/bioloid.xacro (robot description, xacro)
@@ -2,4 +2,11 @@
 <robot xmlns:xacro="http://www.ros.org/wiki/xacro" name="bioloid">
 <!-- Modified Bioloid Comprehensive humanoid, with CM-5 replaced by PC and custom sensors -->
+<!-- ros_control plugin -->
+<gazebo>
+<plugin name="gazebo_ros_control" filename="libgazebo_ros_control.so">
+    <robotNamespace>/</robotNamespace>
+    <robotSimType>gazebo_ros_control/DefaultRobotHWSim</robotSimType>
+</plugin>
+</gazebo>
 <xacro:property name="pi" value="3.14159"/>
 <xacro:property name="cad_dir" value="file:///mnt/STORAGE/Dropbox/Personal/Programming/Bioloid/CAD"/>
@@ -23,4 +30,14 @@
         <limit lower="${-pi}" upper="${pi}" effort="10" velocity="1.0"/>
     </joint>
+    <transmission name="${prefix}_shoulder_swing_joint_tran">
+        <type>transmission_interface/SimpleTransmission</type>
+        <joint name="${prefix}_shoulder_swing_joint">
+            <hardwareInterface>EffortJointInterface</hardwareInterface>
+        </joint>
+        <actuator name="${prefix}_shoulder_swing_joint_motor">
+            <hardwareInterface>EffortJointInterface</hardwareInterface>
+            <mechanicalReduction>1</mechanicalReduction>
+        </actuator>
+    </transmission>
 </xacro:macro>
 <xacro:macro name="shoulder_lateral_joint" params="prefix reflect">
@@ -33,4 +50,14 @@
         <limit lower="${-pi}" upper="${pi}" effort="10" velocity="1.0"/>
     </joint>
+    <transmission name="${prefix}_shoulder_lateral_joint_tran">
+        <type>transmission_interface/SimpleTransmission</type>
+        <joint name="${prefix}_shoulder_lateral_joint">
+            <hardwareInterface>EffortJointInterface</hardwareInterface>
+        </joint>
+        <actuator name="${prefix}_shoulder_lateral_joint_motor">
+            <hardwareInterface>EffortJointInterface</hardwareInterface>
+            <mechanicalReduction>1</mechanicalReduction>
+        </actuator>
+    </transmission>
 </xacro:macro>
 <xacro:macro name="elbow_joint" params="prefix reflect">
@@ -42,4 +69,14 @@
         <limit lower="${-1.77}" upper="${1.77}" effort="10" velocity="1.0"/>
     </joint>
+    <transmission name="${prefix}_elbow_joint_tran">
+        <type>transmission_interface/SimpleTransmission</type>
+        <joint name="${prefix}_elbow_joint">
+            <hardwareInterface>EffortJointInterface</hardwareInterface>
+        </joint>
+        <actuator name="${prefix}_elbow_joint_motor">
+            <hardwareInterface>EffortJointInterface</hardwareInterface>
+            <mechanicalReduction>1</mechanicalReduction>
+        </actuator>
+    </transmission>
 </xacro:macro>
 <xacro:macro name="hand_joint" params="prefix">
@@ -58,4 +95,14 @@
         <limit lower="${-pi/4}" upper="${pi/4}" effort="10" velocity="1.0"/>
     </joint>
+    <transmission name="${prefix}_hip_twist_joint_tran">
+        <type>transmission_interface/SimpleTransmission</type>
+        <joint name="${prefix}_hip_twist_joint">
+            <hardwareInterface>EffortJointInterface</hardwareInterface>
+        </joint>
+        <actuator name="${prefix}_hip_twist_joint_motor">
+            <hardwareInterface>EffortJointInterface</hardwareInterface>
+            <mechanicalReduction>1</mechanicalReduction>
+        </actuator>
+    </transmission>
 </xacro:macro>
 <xacro:macro name="hip_lateral_joint" params="prefix reflect">
@@ -67,4 +114,14 @@
         <limit lower="${-0.3}" upper="${0.3}" effort="10" velocity="1.0"/>
     </joint>
+    <transmission name="${prefix}_hip_lateral_joint_tran">
+        <type>transmission_interface/SimpleTransmission</type>
+        <joint name="${prefix}_hip_lateral_joint">
+            <hardwareInterface>EffortJointInterface</hardwareInterface>
+        </joint>
+        <actuator name="${prefix}_hip_lateral_joint_motor">
+            <hardwareInterface>EffortJointInterface</hardwareInterface>
+            <mechanicalReduction>1</mechanicalReduction>
+        </actuator>
+    </transmission>
 </xacro:macro>
 <xacro:macro name="hip_swing_joint" params="prefix reflect rotatex">
@@ -76,4 +133,14 @@
         <limit lower="${-pi/2}" upper="${pi/2}" effort="10" velocity="1.0"/>
     </joint>
+    <transmission name="${prefix}_hip_swing_joint_tran">
+        <type>transmission_interface/SimpleTransmission</type>
+        <joint name="${prefix}_hip_swing_joint">
+            <hardwareInterface>EffortJointInterface</hardwareInterface>
+        </joint>
+        <actuator name="${prefix}_hip_swing_joint_motor">
+            <hardwareInterface>EffortJointInterface</hardwareInterface>
+            <mechanicalReduction>1</mechanicalReduction>
+        </actuator>
+    </transmission>
 </xacro:macro>
 <xacro:macro name="knee_joint" params="prefix reflect">
@@ -85,4 +152,14 @@
         <limit lower="${-pi}" upper="${0}" effort="10" velocity="1.0"/>
     </joint>
+    <transmission name="${prefix}_knee_joint_tran">
+        <type>transmission_interface/SimpleTransmission</type>
+        <joint name="${prefix}_knee_joint">
+            <hardwareInterface>EffortJointInterface</hardwareInterface>
+        </joint>
+        <actuator name="${prefix}_knee_joint_motor">
+            <hardwareInterface>EffortJointInterface</hardwareInterface>
+            <mechanicalReduction>1</mechanicalReduction>
+        </actuator>
+    </transmission>
 </xacro:macro>
 <xacro:macro name="ankle_swing_joint" params="prefix reflect">
@@ -94,4 +171,14 @@
         <limit lower="${-0.45}" upper="${pi/2}" effort="10" velocity="1.0"/>
     </joint>
+    <transmission name="${prefix}_ankle_swing_joint_tran">
+        <type>transmission_interface/SimpleTransmission</type>
+        <joint name="${prefix}_ankle_swing_joint">
+            <hardwareInterface>EffortJointInterface</hardwareInterface>
+        </joint>
+        <actuator name="${prefix}_ankle_swing_joint_motor">
+            <hardwareInterface>EffortJointInterface</hardwareInterface>
+            <mechanicalReduction>1</mechanicalReduction>
+        </actuator>
+    </transmission>
 </xacro:macro>
 <xacro:macro name="ankle_lateral_joint" params="prefix reflect">
@@ -103,4 +190,14 @@
         <limit lower="${-0.7}" upper="${0.7}" effort="10" velocity="1.0"/>
     </joint>
+    <transmission name="${prefix}_ankle_lateral_joint_tran">
+        <type>transmission_interface/SimpleTransmission</type>
+        <joint name="${prefix}_ankle_lateral_joint">
+            <hardwareInterface>EffortJointInterface</hardwareInterface>
+        </joint>
+        <actuator name="${prefix}_ankle_lateral_joint_motor">
+            <hardwareInterface>EffortJointInterface</hardwareInterface>
+            <mechanicalReduction>1</mechanicalReduction>
+        </actuator>
+    </transmission>
 </xacro:macro>
 <xacro:macro name="foot_joint" params="prefix">
@@ -127,7 +224,7 @@
     </visual>
     <!--<inertial>
-      <origin xyz="0 0 0"/>
-      <mass value="1.0"/>
-      <inertia  ixx="0.001" ixy="0.0"  ixz="0.0"  iyy="0.001"  iyz="0.0"  izz="0.001"/>
+        <origin xyz="0 0 0"/>
+        <mass value="1.0"/>
+        <inertia  ixx="0.001" ixy="0.0"  ixz="0.0"  iyy="0.001"  iyz="0.0"  izz="0.001"/>
     </inertial>-->
 </link>
@@ -156,7 +253,7 @@
     </visual>
     <inertial>
-      <origin xyz="0 0 0"/>
-      <mass value="1.0"/>
-      <inertia  ixx="0.001" ixy="0.0"  ixz="0.0"  iyy="0.001"  iyz="0.0"  izz="0.001"/>
+        <origin xyz="0 0 0"/>
+        <mass value="1.0"/>
+        <inertia  ixx="0.001" ixy="0.0"  ixz="0.0"  iyy="0.001"  iyz="0.0"  izz="0.001"/>
     </inertial>-->
 <!--</link>-->
@@ -199,7 +296,7 @@
     </collision>
     <inertial>
-      <origin xyz="0 0 0"/>
-      <mass value="1.0"/>
-      <inertia  ixx="0.001" ixy="0.0"  ixz="0.0"  iyy="0.001"  iyz="0.0"  izz="0.001"/>
+        <origin xyz="0 0 0"/>
+        <mass value="1.0"/>
+        <inertia  ixx="0.001" ixy="0.0"  ixz="0.0"  iyy="0.001"  iyz="0.0"  izz="0.001"/>
     </inertial>
 </link>
@@ -227,7 +324,7 @@
     </collision>
     <inertial>
-      <origin xyz="0 0 0"/>
-      <mass value="1.0"/>
-      <inertia  ixx="0.001" ixy="0.0"  ixz="0.0"  iyy="0.001"  iyz="0.0"  izz="0.001"/>
+        <origin xyz="0 0 0"/>
+        <mass value="1.0"/>
+        <inertia  ixx="0.001" ixy="0.0"  ixz="0.0"  iyy="0.001"  iyz="0.0"  izz="0.001"/>
     </inertial>
 </link>
@@ -324,7 +421,7 @@
     </collision>
     <inertial>
-      <origin xyz="0 0 0"/>
-      <mass value="1.0"/>
-      <inertia  ixx="0.001" ixy="0.0"  ixz="0.0"  iyy="0.001"  iyz="0.0"  izz="0.001"/>
+        <origin xyz="0 0 0"/>
+        <mass value="1.0"/>
+        <inertia  ixx="0.001" ixy="0.0"  ixz="0.0"  iyy="0.001"  iyz="0.0"  izz="0.001"/>
     </inertial>
 </link>
@@ -343,7 +440,7 @@
     </collision>
     <inertial>
-      <origin xyz="0 0 0"/>
-      <mass value="1.0"/>
-      <inertia  ixx="0.001" ixy="0.0"  ixz="0.0"  iyy="0.001"  iyz="0.0"  izz="0.001"/>
+        <origin xyz="0 0 0"/>
+        <mass value="1.0"/>
+        <inertia  ixx="0.001" ixy="0.0"  ixz="0.0"  iyy="0.001"  iyz="0.0"  izz="0.001"/>
     </inertial>
 </link>
@@ -362,7 +459,7 @@
     </collision>
     <inertial>
-      <origin xyz="0 0 0"/>
-      <mass value="1.0"/>
-      <inertia  ixx="0.001" ixy="0.0"  ixz="0.0"  iyy="0.001"  iyz="0.0"  izz="0.001"/>
+        <origin xyz="0 0 0"/>
+        <mass value="1.0"/>
+        <inertia  ixx="0.001" ixy="0.0"  ixz="0.0"  iyy="0.001"  iyz="0.0"  izz="0.001"/>
     </inertial>
 </link>
@@ -403,7 +500,7 @@
     </collision>
     <inertial>
-      <origin xyz="0 0 0"/>
-      <mass value="1.0"/>
-      <inertia  ixx="0.001" ixy="0.0"  ixz="0.0"  iyy="0.001"  iyz="0.0"  izz="0.001"/>
+        <origin xyz="0 0 0"/>
+        <mass value="1.0"/>
+        <inertia  ixx="0.001" ixy="0.0"  ixz="0.0"  iyy="0.001"  iyz="0.0"  izz="0.001"/>
     </inertial>
 </link>
@@ -444,7 +541,7 @@
     </collision>
     <inertial>
-      <origin xyz="0 0 0"/>
-      <mass value="1.0"/>
-      <inertia  ixx="0.001" ixy="0.0"  ixz="0.0"  iyy="0.001"  iyz="0.0"  izz="0.001"/>
+        <origin xyz="0 0 0"/>
+        <mass value="1.0"/>
+        <inertia  ixx="0.001" ixy="0.0"  ixz="0.0"  iyy="0.001"  iyz="0.0"  izz="0.001"/>
     </inertial>
 </link>
@@ -476,7 +573,7 @@
     </collision>
     <inertial>
-      <origin xyz="0 0 0"/>
-      <mass value="1.0"/>
-      <inertia  ixx="0.001" ixy="0.0"  ixz="0.0"  iyy="0.001"  iyz="0.0"  izz="0.001"/>
+        <origin xyz="0 0 0"/>
+        <mass value="1.0"/>
+        <inertia  ixx="0.001" ixy="0.0"  ixz="0.0"  iyy="0.001"  iyz="0.0"  izz="0.001"/>
     </inertial>
 </link>
@@ -501,7 +598,7 @@
     </collision>
     <inertial>
-      <origin xyz="0 0 0"/>
-      <mass value="1.0"/>
-      <inertia  ixx="0.001" ixy="0.0"  ixz="0.0"  iyy="0.001"  iyz="0.0"  izz="0.001"/>
+        <origin xyz="0 0 0"/>
+        <mass value="1.0"/>
+        <inertia  ixx="0.001" ixy="0.0"  ixz="0.0"  iyy="0.001"  iyz="0.0"  izz="0.001"/>
     </inertial>
 </link>
@@ -533,7 +630,7 @@
     </collision>
     <inertial>
-      <origin xyz="0 0 0"/>
-      <mass value="1.0"/>
-      <inertia  ixx="0.001" ixy="0.0"  ixz="0.0"  iyy="0.001"  iyz="0.0"  izz="0.001"/>
+        <origin xyz="0 0 0"/>
+        <mass value="1.0"/>
+        <inertia  ixx="0.001" ixy="0.0"  ixz="0.0"  iyy="0.001"  iyz="0.0"  izz="0.001"/>
     </inertial>
 </link>
@@ -558,7 +655,7 @@
     </collision>
     <inertial>
-      <origin xyz="0 0 0"/>
-      <mass value="1.0"/>
-      <inertia  ixx="0.001" ixy="0.0"  ixz="0.0"  iyy="0.001"  iyz="0.0"  izz="0.001"/>
+        <origin xyz="0 0 0"/>
+        <mass value="1.0"/>
+        <inertia  ixx="0.001" ixy="0.0"  ixz="0.0"  iyy="0.001"  iyz="0.0"  izz="0.001"/>
     </inertial>
 </link>
@@ -577,7 +674,7 @@
     </collision>
     <inertial>
-      <origin xyz="0 0 0"/>
-      <mass value="1.0"/>
-      <inertia  ixx="0.001" ixy="0.0"  ixz="0.0"  iyy="0.001"  iyz="0.0"  izz="0.001"/>
+        <origin xyz="0 0 0"/>
+        <mass value="1.0"/>
+        <inertia  ixx="0.001" ixy="0.0"  ixz="0.0"  iyy="0.001"  iyz="0.0"  izz="0.001"/>
     </inertial>
 </link>
@@ -596,7 +693,7 @@
     </collision>
     <inertial>
-      <origin xyz="0 0 0"/>
-      <mass value="1.0"/>
-      <inertia  ixx="0.001" ixy="0.0"  ixz="0.0"  iyy="0.001"  iyz="0.0"  izz="0.001"/>
+        <origin xyz="0 0 0"/>
+        <mass value="1.0"/>
+        <inertia  ixx="0.001" ixy="0.0"  ixz="0.0"  iyy="0.001"  iyz="0.0"  izz="0.001"/>
     </inertial>
 </link>
@@ -637,7 +734,7 @@
     </collision>
     <inertial>
-      <origin xyz="0 0 0"/>
-      <mass value="1.0"/>
-      <inertia  ixx="0.001" ixy="0.0"  ixz="0.0"  iyy="0.001"  iyz="0.0"  izz="0.001"/>
+        <origin xyz="0 0 0"/>
+        <mass value="1.0"/>
+        <inertia  ixx="0.001" ixy="0.0"  ixz="0.0"  iyy="0.001"  iyz="0.0"  izz="0.001"/>
     </inertial>
 </link>
@@ -678,7 +775,7 @@
     </collision>
     <inertial>
-      <origin xyz="0 0 0"/>
-      <mass value="1.0"/>
-      <inertia  ixx="0.001" ixy="0.0"  ixz="0.0"  iyy="0.001"  iyz="0.0"  izz="0.001"/>
+        <origin xyz="0 0 0"/>
+        <mass value="1.0"/>
+        <inertia  ixx="0.001" ixy="0.0"  ixz="0.0"  iyy="0.001"  iyz="0.0"  izz="0.001"/>
     </inertial>
 </link>
@@ -707,7 +804,7 @@
     </collision>
     <inertial>
-      <origin xyz="0 0 0"/>
-      <mass value="1.0"/>
-      <inertia  ixx="0.001" ixy="0.0"  ixz="0.0"  iyy="0.001"  iyz="0.0"  izz="0.001"/>
+        <origin xyz="0 0 0"/>
+        <mass value="1.0"/>
+        <inertia  ixx="0.001" ixy="0.0"  ixz="0.0"  iyy="0.001"  iyz="0.0"  izz="0.001"/>
     </inertial>
 </link>
@@ -736,7 +833,7 @@
     </collision>
     <inertial>
-      <origin xyz="0 0 0"/>
-      <mass value="1.0"/>
-      <inertia  ixx="0.001" ixy="0.0"  ixz="0.0"  iyy="0.001"  iyz="0.0"  izz="0.001"/>
+        <origin xyz="0 0 0"/>
+        <mass value="1.0"/>
+        <inertia  ixx="0.001" ixy="0.0"  ixz="0.0"  iyy="0.001"  iyz="0.0"  izz="0.001"/>
     </inertial>
 </link>
@@ -770,7 +867,7 @@
     </collision>
     <inertial>
-      <origin xyz="0 0 0"/>
-      <mass value="1.0"/>
-      <inertia  ixx="0.001" ixy="0.0"  ixz="0.0"  iyy="0.001"  iyz="0.0"  izz="0.001"/>
+        <origin xyz="0 0 0"/>
+        <mass value="1.0"/>
+        <inertia  ixx="0.001" ixy="0.0"  ixz="0.0"  iyy="0.001"  iyz="0.0"  izz="0.001"/>
     </inertial>
 </link>
@@ -804,7 +901,7 @@
     </collision>
     <inertial>
-      <origin xyz="0 0 0"/>
-      <mass value="1.0"/>
-      <inertia  ixx="0.001" ixy="0.0"  ixz="0.0"  iyy="0.001"  iyz="0.0"  izz="0.001"/>
+        <origin xyz="0 0 0"/>
+        <mass value="1.0"/>
+        <inertia  ixx="0.001" ixy="0.0"  ixz="0.0"  iyy="0.001"  iyz="0.0"  izz="0.001"/>
     </inertial>
 </link>
@@ -841,7 +938,7 @@
     </collision>
     <inertial>
-      <origin xyz="0 0 0"/>
-      <mass value="1.0"/>
-      <inertia  ixx="0.001" ixy="0.0"  ixz="0.0"  iyy="0.001"  iyz="0.0"  izz="0.001"/>
+        <origin xyz="0 0 0"/>
+        <mass value="1.0"/>
+        <inertia  ixx="0.001" ixy="0.0"  ixz="0.0"  iyy="0.001"  iyz="0.0"  izz="0.001"/>
     </inertial>
 </link>
@@ -878,7 +975,7 @@
     </collision>
     <inertial>
-      <origin xyz="0 0 0"/>
-      <mass value="1.0"/>
-      <inertia  ixx="0.001" ixy="0.0"  ixz="0.0"  iyy="0.001"  iyz="0.0"  izz="0.001"/>
+        <origin xyz="0 0 0"/>
+        <mass value="1.0"/>
+        <inertia  ixx="0.001" ixy="0.0"  ixz="0.0"  iyy="0.001"  iyz="0.0"  izz="0.001"/>
     </inertial>
 </link>
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
Commit message: Added 3D modeol for USB2AX to URDF. Updated RViz config file.

File: src/bioloid_master/urdf/bioloid.xacro (robot description, xacro)
@@ -277,4 +277,8 @@
         <origin xyz="-0.008 0 0" rpy="${-pi/2} 0 ${-pi/2}"/>
     </visual>
+    <visual>
+        <xacro:default_geometry cad_file="USB2AX-v3.1"/>
+        <origin xyz="-0.0075 -0.0601 -0.001" rpy="0 ${pi/2} 0"/>
+    </visual>
     <collision name="head_bracket_collision">
         <origin xyz="-0.009 0 0"/>
@@ -293,4 +297,10 @@
         <geometry>
             <box size="0.021 0.087 0.058"/>
+        </geometry>
+    </collision>
+    <collision name="usb2ax_collision">
+        <origin xyz="-0.0042 -0.05355 -0.001"/>
+        <geometry>
+            <box size="0.00661 0.037 0.0151"/>
         </geometry>
     </collision>
