Commit message: Split xacro file into logical sub-groups. Individual files for: 1) Main robot links and joints 2) Choice between vanilla Bioloid parts or custom Bioloid parts 3) Gazebo-related elements Updated launch file to include dummy base publisher (for vanilla Bioloid). Removed stand-alone xacro for vanilla Bioloid. Removed URDF files (not needed since URDF files are produced on-the-fly by xacro.py).

File: src/bioloid_master/urdf/bioloid.xacro (robot description, xacro)
@@ -1,1076 +1,767 @@
 <?xml version="1.0"?>
 <robot xmlns:xacro="http://www.ros.org/wiki/xacro" name="bioloid">
-<!-- Modified Bioloid Comprehensive humanoid, with CM-5 replaced by PC and custom sensors -->
-<!-- ros_control plugin -->
-<gazebo>
-<plugin name="gazebo_ros_control" filename="libgazebo_ros_control.so">
-    <robotNamespace>/</robotNamespace>
-    <robotSimType>gazebo_ros_control/DefaultRobotHWSim</robotSimType>
-</plugin>
-</gazebo>
-<xacro:property name="pi" value="3.14159"/>
-<xacro:property name="cad_dir" value="file:///mnt/STORAGE/Dropbox/Personal/Programming/Bioloid/CAD"/>
-<!-- Typically, STL/DAE model units are in mm, but RViz units are in m, hence models must be scaled down by 1000. -->
-<xacro:macro name="default_geometry" params="cad_file suffix:=_FCD-Conv_BDR-Col extension:=dae">
-    <geometry>
-        <mesh filename="${cad_dir}/${cad_file}${suffix}.${extension}" scale="0.001 0.001 0.001"/>
-    </geometry>
-</xacro:macro>
-<xacro:macro name="z_rot">
-    <axis xyz="0 0 1"/>
-</xacro:macro>
-<!-- <xacro:macro name="shoulder_swing_joint" params="prefix reflect x"> -->
-<xacro:macro name="shoulder_swing_joint" params="prefix reflect">
-    <joint name="${prefix}_shoulder_swing_joint" type="revolute">
-        <parent link="torso_link"/>
-        <!-- <origin xyz="${reflect*(-0.032)} 0 0" rpy="0 ${reflect*(-pi/2)} ${x*pi}"/> -->
-        <origin xyz="${reflect*(-0.032)} 0 0" rpy="${reflect*(-pi/2)} 0 ${reflect*(pi/2)}"/>
-        <xacro:z_rot/>
-        <child link="${prefix}_shoulder_swing_link"/>
-        <limit lower="${-pi}" upper="${pi}" effort="10" velocity="1.0"/>
+    <!-- Select one and only one of the following include files -->
+    <!-- 1) Standard parts of Bioloid Comprehensive humanoid with 18 AX-12+ servos, which have been replaced in custom version -->
+    <!--    When using this URDF, ensure a transform from odom to base_link is being published -->
+    <!--<xacro:include filename="$(find bioloid_master)/urdf/bioloid_std_parts.xacro" ns="std_parts"/> -->
+    <!-- 2) Custom parts of modified Bioloid Comprehensive humanoid, with CM-5 replaced by PC and custom sensors -->
+    <!--    When using this URDF, ensure a transform from odom to imu_link is being published -->
+    <xacro:include filename="$(find bioloid_master)/urdf/bioloid_custom_parts.xacro" ns="custom_parts"/>
+    <!-- Import gazebo_ros_control plugin -->
+    <xacro:include filename="$(find bioloid_master)/urdf/bioloid_gazebo.xacro" ns="gazebo"/>
+    <xacro:property name="pi" value="3.14159"/>
+    <xacro:property name="cad_dir" value="file:///mnt/STORAGE/Dropbox/Personal/Programming/Bioloid/CAD"/>
+    <!-- Typically, STL/DAE model units are in mm, but RViz units are in m, hence models must be scaled down by 1000. -->
+    <xacro:macro name="default_geometry" params="cad_file suffix:=_FCD-Conv_BDR-Col extension:=dae">
+        <geometry>
+            <mesh filename="${cad_dir}/${cad_file}${suffix}.${extension}" scale="0.001 0.001 0.001"/>
+        </geometry>
+    </xacro:macro>
+    <xacro:macro name="z_rot">
+        <axis xyz="0 0 1"/>
+    </xacro:macro>
+    <!-- <xacro:macro name="shoulder_swing_joint" params="prefix reflect x"> -->
+    <xacro:macro name="shoulder_swing_joint" params="prefix reflect">
+        <joint name="${prefix}_shoulder_swing_joint" type="revolute">
+            <parent link="torso_link"/>
+            <!-- <origin xyz="${reflect*(-0.032)} 0 0" rpy="0 ${reflect*(-pi/2)} ${x*pi}"/> -->
+            <origin xyz="${reflect*(-0.032)} 0 0" rpy="${reflect*(-pi/2)} 0 ${reflect*(pi/2)}"/>
+            <xacro:z_rot/>
+            <child link="${prefix}_shoulder_swing_link"/>
+            <limit lower="${-pi}" upper="${pi}" effort="10" velocity="1.0"/>
+        </joint>
+    </xacro:macro>
+    <xacro:macro name="shoulder_lateral_joint" params="prefix reflect">
+        <joint name="${prefix}_shoulder_lateral_joint" type="revolute">
+            <parent link="${prefix}_shoulder_swing_link"/>
+            <!-- <origin xyz="${reflect*(-0.014)} 0 ${reflect*0.044}" rpy="${-pi/2} 0 0"/> -->
+            <origin xyz="${reflect*(-0.014)} 0 ${reflect*0.044}" rpy="${-pi/2} ${pi/2} 0"/>
+            <xacro:z_rot/>
+            <child link="${prefix}_upper_arm_link"/>
+            <limit lower="${-pi}" upper="${pi}" effort="10" velocity="1.0"/>
+        </joint>
+    </xacro:macro>
+    <xacro:macro name="elbow_joint" params="prefix reflect">
+        <joint name="${prefix}_elbow_joint" type="revolute">
+            <parent link="${prefix}_upper_arm_link"/>
+            <origin xyz="${reflect*-0.0675} 0 0" rpy="0 0 0"/>
+            <xacro:z_rot/>
+            <child link="${prefix}_lower_arm_link"/>
+            <limit lower="${-1.77}" upper="${1.77}" effort="10" velocity="1.0"/>
+        </joint>
+    </xacro:macro>
+    <xacro:macro name="hand_joint" params="prefix">
+        <joint name="${prefix}_hand_joint" type="fixed">
+            <parent link="${prefix}_lower_arm_link"/>
+            <origin xyz="0 0 0" rpy="0 0 0"/>
+            <child link="${prefix}_hand_link"/>
+        </joint>
+    </xacro:macro>
+    <xacro:macro name="hip_twist_joint" params="prefix reflect rotatex rotatez">
+        <joint name="${prefix}_hip_twist_joint" type="revolute">
+            <parent link="torso_link"/>
+            <origin xyz="${reflect*(-0.033)} 0.016 -0.0655" rpy="${rotatex*pi} 0 ${rotatez*pi}"/>
+            <xacro:z_rot/>
+            <child link="${prefix}_hip_twist_link"/>
+            <limit lower="${-pi/4}" upper="${pi/4}" effort="10" velocity="1.0"/>
+        </joint>
+    </xacro:macro>
+    <xacro:macro name="hip_lateral_joint" params="prefix reflect">
+        <joint name="${prefix}_hip_lateral_joint" type="revolute">
+            <parent link="${prefix}_hip_twist_link"/>
+            <origin xyz="0 -0.0153 ${reflect*0.05}" rpy="${reflect*pi/2} 0 0"/>
+            <xacro:z_rot/>
+            <child link="${prefix}_hip_lateral_link"/>
+            <limit lower="${-0.3}" upper="${0.3}" effort="10" velocity="1.0"/>
+        </joint>
+    </xacro:macro>
+    <xacro:macro name="hip_swing_joint" params="prefix reflect rotatex">
+        <joint name="${prefix}_hip_swing_joint" type="revolute">
+            <parent link="${prefix}_hip_lateral_link"/>
+            <origin xyz="0 0 ${reflect*(-0.032)}" rpy="${rotatex*pi} ${-pi/2} 0"/>
+            <xacro:z_rot/>
+            <child link="${prefix}_upper_leg_link"/>
+            <limit lower="${-pi/2}" upper="${pi/2}" effort="10" velocity="1.0"/>
+        </joint>
+    </xacro:macro>
+    <xacro:macro name="knee_joint" params="prefix reflect">
+        <joint name="${prefix}_knee_joint" type="revolute">
+            <parent link="${prefix}_upper_leg_link"/>
+            <origin xyz="${reflect*0.0145} ${reflect*0.075} 0" rpy="0 0 0"/>
+            <xacro:z_rot/>
+            <child link="${prefix}_lower_leg_link"/>
+            <limit lower="${-pi}" upper="${0}" effort="10" velocity="1.0"/>
+        </joint>
+    </xacro:macro>
+    <xacro:macro name="ankle_swing_joint" params="prefix reflect">
+        <joint name="${prefix}_ankle_swing_joint" type="revolute">
+            <parent link="${prefix}_lower_leg_link"/>
+            <origin xyz="${reflect*-0.0145} ${reflect*0.071} 0" rpy="0 0 0"/>
+            <xacro:z_rot/>
+            <child link="${prefix}_ankle_swing_link"/>
+            <limit lower="${-0.45}" upper="${pi/2}" effort="10" velocity="1.0"/>
+        </joint>
+    </xacro:macro>
+    <xacro:macro name="ankle_lateral_joint" params="prefix reflect">
+        <joint name="${prefix}_ankle_lateral_joint" type="revolute">
+            <parent link="${prefix}_ankle_swing_link"/>
+            <origin xyz="${reflect*0.032} 0 0" rpy="0 ${pi/2} 0"/>
+            <xacro:z_rot/>
+            <child link="${prefix}_ankle_lateral_link"/>
+            <limit lower="${-0.7}" upper="${0.7}" effort="10" velocity="1.0"/>
+        </joint>
+    </xacro:macro>
+    <xacro:macro name="foot_joint" params="prefix">
+        <joint name="${prefix}_foot_joint" type="fixed">
+            <parent link="${prefix}_ankle_lateral_link"/>
+            <origin xyz="0 0 0" rpy="0 0 0"/>
+            <child link="${prefix}_foot_link"/>
+        </joint>
+    </xacro:macro>
+    <!-- Base -->
+    <joint name="base_to_torso_joint" type="fixed">
+        <parent link="base_link"/>
+        <origin xyz="0 0 0" rpy="0 0 ${pi/2}"/>
+        <child link="torso_link"/>
     </joint>
-    <transmission name="${prefix}_shoulder_swing_joint_tran">
-        <type>transmission_interface/SimpleTransmission</type>
-        <joint name="${prefix}_shoulder_swing_joint">
-            <hardwareInterface>EffortJointInterface</hardwareInterface>
-        </joint>
-        <actuator name="${prefix}_shoulder_swing_joint_motor">
-            <hardwareInterface>EffortJointInterface</hardwareInterface>
-            <mechanicalReduction>1</mechanicalReduction>
-        </actuator>
-    </transmission>
-</xacro:macro>
-<xacro:macro name="shoulder_lateral_joint" params="prefix reflect">
-    <joint name="${prefix}_shoulder_lateral_joint" type="revolute">
-        <parent link="${prefix}_shoulder_swing_link"/>
-        <!-- <origin xyz="${reflect*(-0.014)} 0 ${reflect*0.044}" rpy="${-pi/2} 0 0"/> -->
-        <origin xyz="${reflect*(-0.014)} 0 ${reflect*0.044}" rpy="${-pi/2} ${pi/2} 0"/>
-        <xacro:z_rot/>
-        <child link="${prefix}_upper_arm_link"/>
-        <limit lower="${-pi}" upper="${pi}" effort="10" velocity="1.0"/>
-    </joint>
-    <transmission name="${prefix}_shoulder_lateral_joint_tran">
-        <type>transmission_interface/SimpleTransmission</type>
-        <joint name="${prefix}_shoulder_lateral_joint">
-            <hardwareInterface>EffortJointInterface</hardwareInterface>
-        </joint>
-        <actuator name="${prefix}_shoulder_lateral_joint_motor">
-            <hardwareInterface>EffortJointInterface</hardwareInterface>
-            <mechanicalReduction>1</mechanicalReduction>
-        </actuator>
-    </transmission>
-</xacro:macro>
-<xacro:macro name="elbow_joint" params="prefix reflect">
-    <joint name="${prefix}_elbow_joint" type="revolute">
-        <parent link="${prefix}_upper_arm_link"/>
-        <origin xyz="${reflect*-0.0675} 0 0" rpy="0 0 0"/>
-        <xacro:z_rot/>
-        <child link="${prefix}_lower_arm_link"/>
-        <limit lower="${-1.77}" upper="${1.77}" effort="10" velocity="1.0"/>
-    </joint>
-    <transmission name="${prefix}_elbow_joint_tran">
-        <type>transmission_interface/SimpleTransmission</type>
-        <joint name="${prefix}_elbow_joint">
-            <hardwareInterface>EffortJointInterface</hardwareInterface>
-        </joint>
-        <actuator name="${prefix}_elbow_joint_motor">
-            <hardwareInterface>EffortJointInterface</hardwareInterface>
-            <mechanicalReduction>1</mechanicalReduction>
-        </actuator>
-    </transmission>
-</xacro:macro>
-<xacro:macro name="hand_joint" params="prefix">
-    <joint name="${prefix}_hand_joint" type="fixed">
-        <parent link="${prefix}_lower_arm_link"/>
-        <origin xyz="0 0 0" rpy="0 0 0"/>
-        <child link="${prefix}_hand_link"/>
-    </joint>
-</xacro:macro>
-<xacro:macro name="hip_twist_joint" params="prefix reflect rotatex rotatez">
-    <joint name="${prefix}_hip_twist_joint" type="revolute">
-        <parent link="torso_link"/>
-        <origin xyz="${reflect*(-0.033)} 0.016 -0.0655" rpy="${rotatex*pi} 0 ${rotatez*pi}"/>
-        <xacro:z_rot/>
-        <child link="${prefix}_hip_twist_link"/>
-        <limit lower="${-pi/4}" upper="${pi/4}" effort="10" velocity="1.0"/>
-    </joint>
-    <transmission name="${prefix}_hip_twist_joint_tran">
-        <type>transmission_interface/SimpleTransmission</type>
-        <joint name="${prefix}_hip_twist_joint">
-            <hardwareInterface>EffortJointInterface</hardwareInterface>
-        </joint>
-        <actuator name="${prefix}_hip_twist_joint_motor">
-            <hardwareInterface>EffortJointInterface</hardwareInterface>
-            <mechanicalReduction>1</mechanicalReduction>
-        </actuator>
-    </transmission>
-</xacro:macro>
-<xacro:macro name="hip_lateral_joint" params="prefix reflect">
-    <joint name="${prefix}_hip_lateral_joint" type="revolute">
-        <parent link="${prefix}_hip_twist_link"/>
-        <origin xyz="0 -0.0153 ${reflect*0.05}" rpy="${reflect*pi/2} 0 0"/>
-        <xacro:z_rot/>
-        <child link="${prefix}_hip_lateral_link"/>
-        <limit lower="${-0.3}" upper="${0.3}" effort="10" velocity="1.0"/>
-    </joint>
-    <transmission name="${prefix}_hip_lateral_joint_tran">
-        <type>transmission_interface/SimpleTransmission</type>
-        <joint name="${prefix}_hip_lateral_joint">
-            <hardwareInterface>EffortJointInterface</hardwareInterface>
-        </joint>
-        <actuator name="${prefix}_hip_lateral_joint_motor">
-            <hardwareInterface>EffortJointInterface</hardwareInterface>
-            <mechanicalReduction>1</mechanicalReduction>
-        </actuator>
-    </transmission>
-</xacro:macro>
-<xacro:macro name="hip_swing_joint" params="prefix reflect rotatex">
-    <joint name="${prefix}_hip_swing_joint" type="revolute">
-        <parent link="${prefix}_hip_lateral_link"/>
-        <origin xyz="0 0 ${reflect*(-0.032)}" rpy="${rotatex*pi} ${-pi/2} 0"/>
-        <xacro:z_rot/>
-        <child link="${prefix}_upper_leg_link"/>
-        <limit lower="${-pi/2}" upper="${pi/2}" effort="10" velocity="1.0"/>
-    </joint>
-    <transmission name="${prefix}_hip_swing_joint_tran">
-        <type>transmission_interface/SimpleTransmission</type>
-        <joint name="${prefix}_hip_swing_joint">
-            <hardwareInterface>EffortJointInterface</hardwareInterface>
-        </joint>
-        <actuator name="${prefix}_hip_swing_joint_motor">
-            <hardwareInterface>EffortJointInterface</hardwareInterface>
-            <mechanicalReduction>1</mechanicalReduction>
-        </actuator>
-    </transmission>
-</xacro:macro>
-<xacro:macro name="knee_joint" params="prefix reflect">
-    <joint name="${prefix}_knee_joint" type="revolute">
-        <parent link="${prefix}_upper_leg_link"/>
-        <origin xyz="${reflect*0.0145} ${reflect*0.075} 0" rpy="0 0 0"/>
-        <xacro:z_rot/>
-        <child link="${prefix}_lower_leg_link"/>
-        <limit lower="${-pi}" upper="${0}" effort="10" velocity="1.0"/>
-    </joint>
-    <transmission name="${prefix}_knee_joint_tran">
-        <type>transmission_interface/SimpleTransmission</type>
-        <joint name="${prefix}_knee_joint">
-            <hardwareInterface>EffortJointInterface</hardwareInterface>
-        </joint>
-        <actuator name="${prefix}_knee_joint_motor">
-            <hardwareInterface>EffortJointInterface</hardwareInterface>
-            <mechanicalReduction>1</mechanicalReduction>
-        </actuator>
-    </transmission>
-</xacro:macro>
-<xacro:macro name="ankle_swing_joint" params="prefix reflect">
-    <joint name="${prefix}_ankle_swing_joint" type="revolute">
-        <parent link="${prefix}_lower_leg_link"/>
-        <origin xyz="${reflect*-0.0145} ${reflect*0.071} 0" rpy="0 0 0"/>
-        <xacro:z_rot/>
-        <child link="${prefix}_ankle_swing_link"/>
-        <limit lower="${-0.45}" upper="${pi/2}" effort="10" velocity="1.0"/>
-    </joint>
-    <transmission name="${prefix}_ankle_swing_joint_tran">
-        <type>transmission_interface/SimpleTransmission</type>
-        <joint name="${prefix}_ankle_swing_joint">
-            <hardwareInterface>EffortJointInterface</hardwareInterface>
-        </joint>
-        <actuator name="${prefix}_ankle_swing_joint_motor">
-            <hardwareInterface>EffortJointInterface</hardwareInterface>
-            <mechanicalReduction>1</mechanicalReduction>
-        </actuator>
-    </transmission>
-</xacro:macro>
-<xacro:macro name="ankle_lateral_joint" params="prefix reflect">
-    <joint name="${prefix}_ankle_lateral_joint" type="revolute">
-        <parent link="${prefix}_ankle_swing_link"/>
-        <origin xyz="${reflect*0.032} 0 0" rpy="0 ${pi/2} 0"/>
-        <xacro:z_rot/>
-        <child link="${prefix}_ankle_lateral_link"/>
-        <limit lower="${-0.7}" upper="${0.7}" effort="10" velocity="1.0"/>
-    </joint>
-    <transmission name="${prefix}_ankle_lateral_joint_tran">
-        <type>transmission_interface/SimpleTransmission</type>
-        <joint name="${prefix}_ankle_lateral_joint">
-            <hardwareInterface>EffortJointInterface</hardwareInterface>
-        </joint>
-        <actuator name="${prefix}_ankle_lateral_joint_motor">
-            <hardwareInterface>EffortJointInterface</hardwareInterface>
-            <mechanicalReduction>1</mechanicalReduction>
-        </actuator>
-    </transmission>
-</xacro:macro>
-<xacro:macro name="foot_joint" params="prefix">
-    <joint name="${prefix}_foot_joint" type="fixed">
-        <parent link="${prefix}_ankle_lateral_link"/>
-        <origin xyz="0 0 0" rpy="0 0 0"/>
-        <child link="${prefix}_foot_link"/>
-    </joint>
-</xacro:macro>
-<!-- IMU -->
-<joint name="imu_to_base_joint" type="fixed">
-    <parent link="imu_link"/>
-    <origin xyz="0.01 0 0.0788" rpy="0 0 0"/>
-    <child link="base_link"/>
-</joint>
-<link name="imu_link">
-    <visual>
-        <geometry>
-            <box size="0.04 0.02 0.005"/>
-        </geometry>
-        <material name="green">
-            <color rgba="0.0 1.0 0.0 1.0"/>
-        </material>
-    </visual>
-    <!--<inertial>
-        <origin xyz="0 0 0"/>
-        <mass value="1.0"/>
-        <inertia  ixx="0.001" ixy="0.0"  ixz="0.0"  iyy="0.001"  iyz="0.0"  izz="0.001"/>
-    </inertial>-->
-</link>
-<!-- Base -->
-<joint name="base_to_torso_joint" type="fixed">
-    <parent link="base_link"/>
-    <origin xyz="0 0 0" rpy="0 0 ${pi/2}"/>
-    <child link="torso_link"/>
-</joint>
-<link name="base_link">
-</link>
-<!-- Camera -->
-<!--<joint name="camera_joint" type="fixed">
-    <origin xyz="0 0 0.075" rpy="${pi/2} 0 ${pi/2}"/>
-    <parent link="base_link"/>
-    <child link="camera_link"/>
-</joint>
-<link name="camera_link">-->
-    <!--<visual>
-        <geometry>
-            <box size="0.01 0.01 0.01"/>
-        </geometry>
-        <material name="black">
-            <color rgba="0.0 0.0 0.0 1.0"/>
-        </material>
-    </visual>
-    <inertial>
-        <origin xyz="0 0 0"/>
-        <mass value="1.0"/>
-        <inertia  ixx="0.001" ixy="0.0"  ixz="0.0"  iyy="0.001"  iyz="0.0"  izz="0.001"/>
-    </inertial>-->
-<!--</link>-->
-<!-- Head -->
-<joint name="head_joint" type="fixed">
-    <origin xyz="0 0 0.058" rpy="0 0 0"/>
-    <parent link="base_link"/>
-    <child link="head_link"/>
-</joint>
-<link name="head_link">
-    <visual>
-        <xacro:default_geometry cad_file="FP04-F5"/>
-        <origin xyz="0 0 0" rpy="${pi/2} 0 ${-pi/2}"/>
-    </visual>
-    <visual>
-        <xacro:default_geometry cad_file="FP04-F10"/>
-        <origin xyz="0 0 -0.0342" rpy="${pi/2} 0 ${-pi/2}"/>
-    </visual>
-    <visual>
-        <xacro:default_geometry cad_file="RaspPiB_plus_3d_step_V10" suffix="_FCD-Conv"/>
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
Commit message: Moved CAD files into repo. Changed CAD file to relative path in Xacro file.

File: src/bioloid_master/urdf/bioloid.xacro (robot description, xacro)
@@ -11,5 +11,5 @@
     <xacro:include filename="$(find bioloid_master)/urdf/bioloid_gazebo.xacro" ns="gazebo"/>
     <xacro:property name="pi" value="3.14159"/>
-    <xacro:property name="cad_dir" value="file:///mnt/STORAGE/Dropbox/Personal/Programming/Bioloid/CAD"/>
+    <xacro:property name="cad_dir" value="file://$(find bioloid_master)/../../assets/cad"/>
     <!-- Typically, STL/DAE model units are in mm, but RViz units are in m, hence models must be scaled down by 1000. -->
     <xacro:macro name="default_geometry" params="cad_file suffix:=_FCD-Conv_BDR-Col extension:=dae">
