Commit message: Centred feet to make space for FSRs connections on the actual robot. Added FSR CAD parts to customised model. Original configuration preserved for standard model.

File: src/bioloid_master/urdf/bioloid.xacro (robot description, xacro)
@@ -729,39 +729,5 @@
     <!-- Right ankle lateral to foot -->
     <xacro:foot_joint prefix="right"/>
-    <link name="right_foot_link">
-        <visual>
-            <xacro:default_geometry cad_file="FP04-F12"/>
-            <origin xyz="-0.008 0.0235 -0.016" rpy="0 ${-pi/2} 0"/>
-        </visual>
-        <collision name="right_foot_collision">
-            <origin xyz="-0.008 0.0277 -0.016"/>
-            <geometry>
-                <box size="0.061 0.009 0.101"/>
-            </geometry>
-        </collision>
-        <inertial>
-            <origin xyz="0 0 0"/>
-            <mass value="1.0"/>
-            <inertia  ixx="0.001" ixy="0.0"  ixz="0.0"  iyy="0.001"  iyz="0.0"  izz="0.001"/>
-        </inertial>
-    </link>
     <!-- Left ankle lateral to foot -->
     <xacro:foot_joint prefix="left"/>
-    <link name="left_foot_link">
-        <visual>
-            <xacro:default_geometry cad_file="FP04-F12"/>
-            <origin xyz="0.008 -0.0235 0.016" rpy="${pi} ${pi/2} 0"/>
-        </visual>
-        <collision name="left_foot_collision">
-            <origin xyz="0.008 -0.0277 0.016"/>
-            <geometry>
-                <box size="0.061 0.009 0.101"/>
-            </geometry>
-        </collision>
-        <inertial>
-            <origin xyz="0 0 0"/>
-            <mass value="1.0"/>
-            <inertia  ixx="0.001" ixy="0.0"  ixz="0.0"  iyy="0.001"  iyz="0.0"  izz="0.001"/>
-        </inertial>
-    </link>
 </robot>

File: src/bioloid_master/urdf/bioloid_custom_parts.xacro (robot description, xacro)
@@ -215,3 +215,69 @@
         </inertial>
     </link>
+    <!-- Right foot -->
+    <link name="right_foot_link">
+        <visual>
+            <xacro:default_geometry cad_file="FP04-F12"/>
+            <origin xyz="0 0.0235 -0.016" rpy="0 ${-pi/2} 0"/>
+        </visual>
+        <!-- FSR 0 -->
+        <visual>
+            <xacro:default_geometry cad_file="34-47021_FSR_400_Short_Tail"/>
+            <origin xyz="0.022 0.0319 -0.039" rpy="${pi} 0 0"/>
+        </visual>
+        <!-- FSR 1 -->
+        <visual>
+            <xacro:default_geometry cad_file="34-47021_FSR_400_Short_Tail"/>
+            <origin xyz="-0.022 0.0319 -0.039" rpy="${pi} 0 0"/>
+        </visual>
+        <!-- FSR 2 -->
+        <visual>
+            <xacro:default_geometry cad_file="34-47021_FSR_400_Short_Tail"/>
+            <origin xyz="-0.022 0.0319 0.007" rpy="${pi} ${pi} 0"/>
+        </visual>
+        <collision name="right_foot_collision">
+            <origin xyz="0 0.0277 -0.016"/>
+            <geometry>
+                <box size="0.061 0.009 0.101"/>
+            </geometry>
+        </collision>
+        <inertial>
+            <origin xyz="0 0 0"/>
+            <mass value="1.0"/>
+            <inertia  ixx="0.001" ixy="0.0"  ixz="0.0"  iyy="0.001"  iyz="0.0"  izz="0.001"/>
+        </inertial>
+    </link>
+    <!-- Left foot -->
+    <link name="left_foot_link">
+        <visual>
+            <xacro:default_geometry cad_file="FP04-F12"/>
+            <origin xyz="0 -0.0235 0.016" rpy="${pi} ${pi/2} 0"/>
+        </visual>
+        <!-- FSR 3 -->
+        <visual>
+            <xacro:default_geometry cad_file="34-47021_FSR_400_Short_Tail"/>
+            <origin xyz="-0.022 -0.0319 0.039" rpy="0 0 0"/>
+        </visual>
+        <!-- FSR 4 -->
+        <visual>
+            <xacro:default_geometry cad_file="34-47021_FSR_400_Short_Tail"/>
+            <origin xyz="0.022 -0.0319 0.039" rpy="0 0 0"/>
+        </visual>
+        <!-- FSR 5 -->
+        <visual>
+            <xacro:default_geometry cad_file="34-47021_FSR_400_Short_Tail"/>
+            <origin xyz="0.022 -0.0319 -0.007" rpy="0 ${pi} 0"/>
+        </visual>
+        <collision name="left_foot_collision">
+            <origin xyz="0 -0.0277 0.016"/>
+            <geometry>
+                <box size="0.061 0.009 0.101"/>
+            </geometry>
+        </collision>
+        <inertial>
+            <origin xyz="0 0 0"/>
+            <mass value="1.0"/>
+            <inertia  ixx="0.001" ixy="0.0"  ixz="0.0"  iyy="0.001"  iyz="0.0"  izz="0.001"/>
+        </inertial>
+    </link>
 </robot>

File: src/bioloid_master/urdf/bioloid_std_parts.xacro (robot description, xacro)
@@ -81,3 +81,39 @@
         </inertial>
     </link>
+    <!-- Right foot -->
+    <link name="right_foot_link">
+        <visual>
+            <xacro:default_geometry cad_file="FP04-F12"/>
+            <origin xyz="-0.008 0.0235 -0.016" rpy="0 ${-pi/2} 0"/>
+        </visual>
+        <collision name="right_foot_collision">
+            <origin xyz="-0.008 0.0277 -0.016"/>
+            <geometry>
+                <box size="0.061 0.009 0.101"/>
+            </geometry>
+        </collision>
+        <inertial>
+            <origin xyz="0 0 0"/>
+            <mass value="1.0"/>
+            <inertia  ixx="0.001" ixy="0.0"  ixz="0.0"  iyy="0.001"  iyz="0.0"  izz="0.001"/>
+        </inertial>
+    </link>
+    <!-- Left foot -->
+    <link name="left_foot_link">
+        <visual>
+            <xacro:default_geometry cad_file="FP04-F12"/>
+            <origin xyz="0.008 -0.0235 0.016" rpy="${pi} ${pi/2} 0"/>
+        </visual>
+        <collision name="left_foot_collision">
+            <origin xyz="0.008 -0.0277 0.016"/>
+            <geometry>
+                <box size="0.061 0.009 0.101"/>
+            </geometry>
+        </collision>
+        <inertial>
+            <origin xyz="0 0 0"/>
+            <mass value="1.0"/>
+            <inertia  ixx="0.001" ixy="0.0"  ixz="0.0"  iyy="0.001"  iyz="0.0"  izz="0.001"/>
+        </inertial>
+    </link>
 </robot>

Commit message: Xacro updates for ROS Kinetic compatibility

File: src/bioloid_master/urdf/bioloid.xacro (robot description, xacro)
@@ -1,4 +1,16 @@
 <?xml version="1.0"?>
 <robot xmlns:xacro="http://www.ros.org/wiki/xacro" name="bioloid">
+    <!-- Pi is now predefined -->
+    <!-- <xacro:property name="pi" value="3.14159"/> -->
+    <xacro:property name="cad_dir" value="file://$(find bioloid_master)/../../assets/cad"/>
+    <!-- Typically, STL/DAE model units are in mm, but RViz units are in m, hence models must be scaled down by 1000. -->
+    <xacro:macro name="default_geometry" params="cad_file suffix:=_FCD-Conv_BDR-Col extension:=dae">
+        <geometry>
+            <mesh filename="${cad_dir}/${cad_file}${suffix}.${extension}" scale="0.001 0.001 0.001"/>
+        </geometry>
+    </xacro:macro>
+    <xacro:macro name="z_rot">
+        <axis xyz="0 0 1"/>
+    </xacro:macro>
     <!-- Select one and only one of the following include files -->
     <!-- 1) Standard parts of Bioloid Comprehensive humanoid with 18 AX-12+ servos, which have been replaced in custom version -->
@@ -7,18 +19,7 @@
     <!-- 2) Custom parts of modified Bioloid Comprehensive humanoid, with CM-5 replaced by PC and custom sensors -->
     <!--    When using this URDF, ensure a transform from odom to imu_link is being published -->
-    <xacro:include filename="$(find bioloid_master)/urdf/bioloid_custom_parts.xacro" ns="custom_parts"/>
+    <xacro:include filename="$(find bioloid_master)/urdf/bioloid_custom_parts.xacro"/>
     <!-- Import gazebo_ros_control plugin -->
-    <xacro:include filename="$(find bioloid_master)/urdf/bioloid_gazebo.xacro" ns="gazebo"/>
-    <xacro:property name="pi" value="3.14159"/>
-    <xacro:property name="cad_dir" value="file://$(find bioloid_master)/../../assets/cad"/>
-    <!-- Typically, STL/DAE model units are in mm, but RViz units are in m, hence models must be scaled down by 1000. -->
-    <xacro:macro name="default_geometry" params="cad_file suffix:=_FCD-Conv_BDR-Col extension:=dae">
-        <geometry>
-            <mesh filename="${cad_dir}/${cad_file}${suffix}.${extension}" scale="0.001 0.001 0.001"/>
-        </geometry>
-    </xacro:macro>
-    <xacro:macro name="z_rot">
-        <axis xyz="0 0 1"/>
-    </xacro:macro>
+    <xacro:include filename="$(find bioloid_master)/urdf/bioloid_gazebo.xacro"/>
     <!-- <xacro:macro name="shoulder_swing_joint" params="prefix reflect x"> -->
     <xacro:macro name="shoulder_swing_joint" params="prefix reflect">

File: src/bioloid_master/urdf/bioloid_gazebo.xacro (robot description, xacro)
@@ -33,4 +33,16 @@
     </xacro:macro>
     <xacro:macro name="elbow_joint_gazebo" params="prefix">
+        <transmission name="${prefix}_elbow_joint_tran">
+            <type>transmission_interface/SimpleTransmission</type>
+            <joint name="${prefix}_elbow_joint">
+                <hardwareInterface>EffortJointInterface</hardwareInterface>
+            </joint>
+            <actuator name="${prefix}_elbow_joint_motor">
+                <hardwareInterface>EffortJointInterface</hardwareInterface>
+                <mechanicalReduction>1</mechanicalReduction>
+            </actuator>
+        </transmission>
+    </xacro:macro>
+    <xacro:macro name="hand_joint_gazebo" params="prefix">
         <transmission name="${prefix}_elbow_joint_tran">
             <type>transmission_interface/SimpleTransmission</type>
@@ -116,25 +128,37 @@
         </transmission>
     </xacro:macro>
-    <xacro:shoulder_swing_joint_gazebo prefix="right"/>
-    <xacro:shoulder_swing_joint_gazebo prefix="left"/>
-    <xacro:shoulder_lateral_joint_gazebo prefix="right"/>
-    <xacro:shoulder_lateral_joint_gazebo prefix="left"/>
-    <xacro:elbow_joint_gazebo prefix="right"/>
-    <xacro:elbow_joint_gazebo prefix="left"/>
-    <xacro:hand_joint_gazebo prefix="right"/>
-    <xacro:hand_joint_gazebo prefix="left"/>
-    <xacro:hip_twist_joint_gazebo prefix="right"/>
-    <xacro:hip_twist_joint_gazebo prefix="left"/>
-    <xacro:hip_lateral_joint_gazebo prefix="right"/>
-    <xacro:hip_lateral_joint_gazebo prefix="left"/>
-    <xacro:hip_swing_joint_gazebo prefix="right"/>
-    <xacro:hip_swing_joint_gazebo prefix="left"/>
-    <xacro:knee_joint_gazebo prefix="right"/>
-    <xacro:knee_joint_gazebo prefix="left"/>
-    <xacro:ankle_swing_joint_gazebo prefix="right"/>
-    <xacro:ankle_swing_joint_gazebo prefix="left"/>
-    <xacro:ankle_lateral_joint_gazebo prefix="right"/>
-    <xacro:ankle_lateral_joint_gazebo prefix="left"/>
-    <xacro:foot_joint_gazebo prefix="right"/>
-    <xacro:foot_joint_gazebo prefix="left"/>
+    <xacro:macro name="foot_joint_gazebo" params="prefix">
+        <transmission name="${prefix}_ankle_lateral_joint_tran">
+            <type>transmission_interface/SimpleTransmission</type>
+            <joint name="${prefix}_ankle_lateral_joint">
+                <hardwareInterface>EffortJointInterface</hardwareInterface>
+            </joint>
+            <actuator name="${prefix}_ankle_lateral_joint_motor">
+                <hardwareInterface>EffortJointInterface</hardwareInterface>
+                <mechanicalReduction>1</mechanicalReduction>
+            </actuator>
+        </transmission>
+    </xacro:macro>
+    <shoulder_swing_joint_gazebo prefix="right"/>
+    <shoulder_swing_joint_gazebo prefix="left"/>
+    <shoulder_lateral_joint_gazebo prefix="right"/>
+    <shoulder_lateral_joint_gazebo prefix="left"/>
+    <elbow_joint_gazebo prefix="right"/>
+    <elbow_joint_gazebo prefix="left"/>
+    <hand_joint_gazebo prefix="right"/>
+    <hand_joint_gazebo prefix="left"/>
+    <hip_twist_joint_gazebo prefix="right"/>
+    <hip_twist_joint_gazebo prefix="left"/>
+    <hip_lateral_joint_gazebo prefix="right"/>
+    <hip_lateral_joint_gazebo prefix="left"/>
+    <hip_swing_joint_gazebo prefix="right"/>
+    <hip_swing_joint_gazebo prefix="left"/>
+    <knee_joint_gazebo prefix="right"/>
+    <knee_joint_gazebo prefix="left"/>
+    <ankle_swing_joint_gazebo prefix="right"/>
+    <ankle_swing_joint_gazebo prefix="left"/>
+    <ankle_lateral_joint_gazebo prefix="right"/>
+    <ankle_lateral_joint_gazebo prefix="left"/>
+    <foot_joint_gazebo prefix="right"/>
+    <foot_joint_gazebo prefix="left"/>
 </robot>
